Commit message: change mesh object file path
Signed-off-by: NaokiTakahashi <naoki.takahashi060@gmail.com>

File: robots/go1_description/models/urdf/depthCamera.xacro (robot description, xacro)
@@ -17,5 +17,5 @@
             <origin xyz="0 0 0" rpy="0 0 0"/>
             <geometry>
-                <mesh filename="package://go1_description/meshes/depthCamera.dae" scale="1 1 1"/>
+                <mesh filename="package://go1_description/models/meshes/depthCamera.dae" scale="1 1 1"/>
             </geometry>
             </visual>

File: robots/go1_description/models/urdf/leg.xacro (robot description, xacro)
@@ -1,5 +1,5 @@
 <?xml version="1.0"?>
 <robot xmlns:xacro="http://www.ros.org/wiki/xacro">
-    <xacro:include filename="$(find go1_description)/xacro/transmission.xacro"/>
+    <xacro:include filename="$(find go1_description)/models/urdf/transmission.xacro"/>
     <xacro:macro name="leg" params="name mirror mirror_dae front_hind front_hind_dae *origin">
         <joint name="${name}_hip_joint" type="revolute">
@@ -31,5 +31,5 @@
                 </xacro:if>
                 <geometry>
-                    <mesh filename="package://go1_description/meshes/hip.dae" scale="1 1 1"/>
+                    <mesh filename="package://go1_description/models/meshes/hip.dae" scale="1 1 1"/>
                 </geometry>
                 <!-- <material name="orange"/> -->
@@ -77,8 +77,8 @@
                 <geometry>
                     <xacro:if value="${mirror_dae == True}">
-                        <mesh filename="package://go1_description/meshes/thigh.dae" scale="1 1 1"/>
+                        <mesh filename="package://go1_description/models/meshes/thigh.dae" scale="1 1 1"/>
                     </xacro:if>
                     <xacro:if value="${mirror_dae == False}">
-                        <mesh filename="package://go1_description/meshes/thigh_mirror.dae" scale="1 1 1"/>
+                        <mesh filename="package://go1_description/models/meshes/thigh_mirror.dae" scale="1 1 1"/>
                     </xacro:if>
                 </geometry>
@@ -112,5 +112,5 @@
                 <origin rpy="0 0 0" xyz="0 0 0"/>
                 <geometry>
-                    <mesh filename="package://go1_description/meshes/calf.dae" scale="1 1 1"/>
+                    <mesh filename="package://go1_description/models/meshes/calf.dae" scale="1 1 1"/>
                 </geometry>
                 <!-- <material name="orange"/> -->

File: robots/go1_description/models/urdf/robot.xacro (robot description, xacro)
@@ -1,11 +1,11 @@
 <?xml version="1.0"?>
 <robot name="go1_description" xmlns:xacro="http://www.ros.org/wiki/xacro">
-    <xacro:include filename="$(find go1_description)/xacro/const.xacro"/>
-    <xacro:include filename="$(find go1_description)/xacro/materials.xacro"/>
-    <xacro:include filename="$(find go1_description)/xacro/leg.xacro"/>
-    <!-- <xacro:include filename="$(find go1_description)/xacro/stairs.xacro"/> -->
-    <xacro:include filename="$(find go1_description)/xacro/gazebo.xacro"/>
-    <xacro:include filename="$(find go1_description)/xacro/depthCamera.xacro"/>
-    <xacro:include filename="$(find go1_description)/xacro/ultraSound.xacro"/>
+    <xacro:include filename="$(find go1_description)/models/urdf/const.xacro"/>
+    <xacro:include filename="$(find go1_description)/models/urdf/materials.xacro"/>
+    <xacro:include filename="$(find go1_description)/models/urdf/leg.xacro"/>
+    <!-- <xacro:include filename="$(find go1_description)/models/urdf/stairs.xacro"/> -->
+    <xacro:include filename="$(find go1_description)/models/urdf/gazebo.xacro"/>
+    <xacro:include filename="$(find go1_description)/models/urdf/depthCamera.xacro"/>
+    <xacro:include filename="$(find go1_description)/models/urdf/ultraSound.xacro"/>
     <!-- <xacro:include filename="$(find go1_gazebo)/launch/stairs.urdf.xacro"/> -->
     <!-- <xacro:stairs stairs="15" xpos="0" ypos="0" zpos="0" /> -->
@@ -13,4 +13,5 @@
     <xacro:property name="rolloverProtection" value="false"/>
     <!-- Debug mode will hung up the robot, use "true" or "false" to switch it. -->
+    <xacro:arg name="DEBUG" default="false"/>
     <xacro:if value="$(arg DEBUG)">
         <link name="world"/>
@@ -38,5 +39,5 @@
             <origin rpy="0 0 0" xyz="0 0 0"/>
             <geometry>
-                <mesh filename="package://go1_description/meshes/trunk.dae" scale="1 1 1"/>
+                <mesh filename="package://go1_description/models/meshes/trunk.dae" scale="1 1 1"/>
             </geometry>
             <!-- <material name="orange"/> -->

File: robots/go1_description/models/urdf/ultraSound.xacro (robot description, xacro)
@@ -17,5 +17,5 @@
             <origin xyz="0 0 0" rpy="0 0 0"/>
             <geometry>
-                <mesh filename="package://go1_description/meshes/ultraSound.dae" scale="1 1 1"/>
+                <mesh filename="package://go1_description/models/meshes/ultraSound.dae" scale="1 1 1"/>
             </geometry>
             <material name="black"/>

Commit message: update link colors
Signed-off-by: NaokiTakahashi <naoki.takahashi060@gmail.com>

File: robots/go1_description/models/urdf/depthCamera.xacro (robot description, xacro)
@@ -19,4 +19,5 @@
           <mesh filename="package://go1_description/models/meshes/depthCamera.dae" scale="1 1 1"/>
         </geometry>
+        <material name="black"/>
       </visual>
       <inertial>

File: robots/go1_description/models/urdf/gazebo.xacro (robot description, xacro)
@@ -152,5 +152,4 @@
   </xacro:if>
   <gazebo reference="base_link">
-    <material>Gazebo/Green</material>
     <turnGravityOff>false</turnGravityOff>
   </gazebo>
@@ -164,10 +163,8 @@
     <mu1>0.2</mu1>
     <mu2>0.2</mu2>
-    <material>Gazebo/White</material>
   </gazebo>
   <gazebo reference="imu_link">
     <mu1>0.2</mu1>
     <mu2>0.2</mu2>
-    <material>Gazebo/Red</material>
   </gazebo>
   <!-- FL leg -->
@@ -175,5 +172,4 @@
     <mu1>0.2</mu1>
     <mu2>0.2</mu2>
-    <material>Gazebo/DarkGrey</material>
   </gazebo>
   <gazebo reference="FL_thigh">
@@ -181,5 +177,4 @@
     <mu2>0.2</mu2>
     <self_collide>1</self_collide>
-    <material>Gazebo/DarkGrey</material>
     <kp value="1000000.0"/>
     <kd value="1.0"/>
@@ -194,5 +189,4 @@
     <mu2>0.6</mu2>
     <self_collide>1</self_collide>
-    <material>Gazebo/DarkGrey</material>
     <kp value="1000000.0"/>
     <kd value="1.0"/>
@@ -202,5 +196,4 @@
     <mu1>0.2</mu1>
     <mu2>0.2</mu2>
-    <material>Gazebo/DarkGrey</material>
   </gazebo>
   <gazebo reference="FR_thigh">
@@ -208,5 +201,4 @@
     <mu2>0.2</mu2>
     <self_collide>1</self_collide>
-    <material>Gazebo/DarkGrey</material>
     <kp value="1000000.0"/>
     <kd value="1.0"/>
@@ -221,5 +213,4 @@
     <mu2>0.6</mu2>
     <self_collide>1</self_collide>
-    <material>Gazebo/DarkGrey</material>
     <kp value="1000000.0"/>
     <kd value="1.0"/>
@@ -229,5 +220,4 @@
     <mu1>0.2</mu1>
     <mu2>0.2</mu2>
-    <material>Gazebo/DarkGrey</material>
   </gazebo>
   <gazebo reference="RL_thigh">
@@ -235,5 +225,4 @@
     <mu2>0.2</mu2>
     <self_collide>1</self_collide>
-    <material>Gazebo/DarkGrey</material>
     <kp value="1000000.0"/>
     <kd value="1.0"/>
@@ -248,5 +237,4 @@
     <mu2>0.6</mu2>
     <self_collide>1</self_collide>
-    <material>Gazebo/DarkGrey</material>
     <kp value="1000000.0"/>
     <kd value="1.0"/>
@@ -256,5 +244,4 @@
     <mu1>0.2</mu1>
     <mu2>0.2</mu2>
-    <material>Gazebo/DarkGrey</material>
   </gazebo>
   <gazebo reference="RR_thigh">
@@ -262,5 +249,4 @@
     <mu2>0.2</mu2>
     <self_collide>1</self_collide>
-    <material>Gazebo/DarkGrey</material>
     <kp value="1000000.0"/>
     <kd value="1.0"/>
@@ -275,5 +261,4 @@
     <mu2>0.6</mu2>
     <self_collide>1</self_collide>
-    <material>Gazebo/DarkGrey</material>
     <kp value="1000000.0"/>
     <kd value="1.0"/>

File: robots/go1_description/models/urdf/leg.xacro (robot description, xacro)
@@ -33,5 +33,5 @@
           <mesh filename="package://go1_description/models/meshes/hip.dae" scale="1 1 1"/>
         </geometry>
-        <!-- <material name="orange"/> -->
+        <material name="silver"/>
       </visual>
       <collision>
@@ -80,5 +80,5 @@
           </xacro:if>
         </geometry>
-        <!-- <material name="orange"/> -->
+        <material name="silver"/>
       </visual>
       <collision>
@@ -108,5 +108,5 @@
           <mesh filename="package://go1_description/models/meshes/calf.dae" scale="1 1 1"/>
         </geometry>
-        <!-- <material name="orange"/> -->
+        <material name="silver"/>
       </visual>
       <collision>
@@ -133,5 +133,5 @@
           <sphere radius="${foot_radius-0.01}"/>
         </geometry>
-        <!-- <material name="orange"/> -->
+        <material name="silver"/>
       </visual>
       <collision>

File: robots/go1_description/models/urdf/unitree_go1.urdf.xacro (robot description, xacro)
@@ -41,5 +41,5 @@
         <mesh filename="package://go1_description/models/meshes/trunk.dae" scale="1 1 1"/>
       </geometry>
-      <!-- <material name="orange"/> -->
+      <material name="silver"/>
     </visual>
     <collision>
@@ -67,5 +67,5 @@
         </geometry>
         <origin rpy="0 0 0" xyz="0 0 0"/>
-        <!-- <material name="white"/> -->
+        <material name="silver"/>
       </visual>
       <collision>
@@ -97,5 +97,5 @@
         <box size="0.001 0.001 0.001"/>
       </geometry>
-      <!-- <material name="red"/> -->
+      <material name="black"/>
     </visual>
     <collision>
