Commit message: add ignition_gazebo flag
Signed-off-by: NaokiTakahashi <naoki.takahashi060@gmail.com>

File: robots/go1_description/models/urdf/const.xacro (robot description, xacro)
@@ -1,4 +1,4 @@
 <?xml version="1.0"?>
-<robot xmlns:xacro="http://www.ros.org/wiki/xacro" name="go1_description">
+<robot xmlns:xacro="http://www.ros.org/wiki/xacro" name="unitree_go1">
   <!-- Constants for robot dimensions -->
   <xacro:property name="PI" value="3.1415926535897931"/>

File: robots/go1_description/models/urdf/depthCamera.xacro (robot description, xacro)
@@ -49,29 +49,31 @@
           </clip>
         </camera>
-        <plugin name="camera_${name}_controller" filename="libgazebo_ros_openni_kinect.so">
-          <baseline>0.025</baseline>
-          <alwaysOn>true</alwaysOn>
-          <updateRate>0.0</updateRate>
-          <cameraName>camera_${name}_ir</cameraName>
-          <imageTopicName>/camera_${name}/color/image_raw</imageTopicName>
-          <cameraInfoTopicName>/camera_${name}/color/camera_info</cameraInfoTopicName>
-          <depthImageTopicName>/camera_${name}/depth/image_raw</depthImageTopicName>
-          <depthImageInfoTopicName>/camera_${name}/depth/camera_info</depthImageInfoTopicName>
-          <!-- <pointCloudTopicName>/camera_${name}/depth/points</pointCloudTopicName> -->
-          <pointCloudTopicName>/cam${camID}/point_cloud_${name}</pointCloudTopicName>
-          <frameName>camera_optical_${name}</frameName>
-          <pointCloudCutoff>0.1</pointCloudCutoff>
-          <pointCloudCutoffMax>1.5</pointCloudCutoffMax>
-          <distortionK1>0.0</distortionK1>
-          <distortionK2>0.0</distortionK2>
-          <distortionK3>0.0</distortionK3>
-          <distortionT1>0.0</distortionT1>
-          <distortionT2>0.0</distortionT2>
-          <CxPrime>0</CxPrime>
-          <Cx>0.0045</Cx>
-          <Cy>0.0039</Cy>
-          <focalLength>0</focalLength>
-          <hackBaseline>0</hackBaseline>
-        </plugin>
+        <xacro:if value="${'$(arg ignition_gazebo)' == 'false'}">
+          <plugin name="camera_${name}_controller" filename="libgazebo_ros_openni_kinect.so">
+            <baseline>0.025</baseline>
+            <alwaysOn>true</alwaysOn>
+            <updateRate>0.0</updateRate>
+            <cameraName>camera_${name}_ir</cameraName>
+            <imageTopicName>/camera_${name}/color/image_raw</imageTopicName>
+            <cameraInfoTopicName>/camera_${name}/color/camera_info</cameraInfoTopicName>
+            <depthImageTopicName>/camera_${name}/depth/image_raw</depthImageTopicName>
+            <depthImageInfoTopicName>/camera_${name}/depth/camera_info</depthImageInfoTopicName>
+            <!-- <pointCloudTopicName>/camera_${name}/depth/points</pointCloudTopicName> -->
+            <pointCloudTopicName>/cam${camID}/point_cloud_${name}</pointCloudTopicName>
+            <frameName>camera_optical_${name}</frameName>
+            <pointCloudCutoff>0.1</pointCloudCutoff>
+            <pointCloudCutoffMax>1.5</pointCloudCutoffMax>
+            <distortionK1>0.0</distortionK1>
+            <distortionK2>0.0</distortionK2>
+            <distortionK3>0.0</distortionK3>
+            <distortionT1>0.0</distortionT1>
+            <distortionT2>0.0</distortionT2>
+            <CxPrime>0</CxPrime>
+            <Cx>0.0045</Cx>
+            <Cy>0.0039</Cy>
+            <focalLength>0</focalLength>
+            <hackBaseline>0</hackBaseline>
+          </plugin>
+        </xacro:if>
       </sensor>
     </gazebo>

File: robots/go1_description/models/urdf/gazebo.xacro (robot description, xacro)
@@ -1,39 +1,47 @@
 <?xml version="1.0"?>
 <robot xmlns:xacro="http://www.ros.org/wiki/xacro">
-  <!-- ros_control plugin -->
-  <gazebo>
-    <plugin name="gazebo_ros_control" filename="libgazebo_ros_control.so">
-      <robotNamespace>/go1_gazebo</robotNamespace>
-      <robotSimType>gazebo_ros_control/DefaultRobotHWSim</robotSimType>
-    </plugin>
-  </gazebo>
-  <!-- Show the trajectory of trunk center. -->
-  <gazebo>
-    <plugin name="3dplot" filename="libLinkPlot3DPlugin.so">
-      <frequency>10</frequency>
-      <plot>
-        <link>base</link>
-        <pose>0 0 0 0 0 0</pose>
-        <material>Gazebo/Yellow</material>
-      </plot>
-    </plugin>
-  </gazebo>
-  <!-- Show the trajectory of foot. You can add another trajectory about another foot. -->
-  <!-- <gazebo>
-        <plugin name="3dplot" filename="libLinkPlot3DPlugin.so">
-            <frequency>100</frequency>
-            <plot>
-                <link>FL_foot</link>
-                <pose>0 0 0 0 0 0</pose>
-                <material>Gazebo/Green</material>
-            </plot>
-        </plugin>
-    </gazebo> -->
-  <gazebo>
-    <plugin filename="libgazebo_ros_force.so" name="gazebo_ros_force">
-      <bodyName>trunk</bodyName>
-      <topicName>/apply_force/trunk</topicName>
-    </plugin>
-  </gazebo>
+  <xacro:arg name="ignition_gazebo" default="true"/>
+  <xacro:if value="$(arg ignition_gazebo)">
+    <gazebo>
+      <plugin filename="ignition-gazebo-joint-state-publisher-system" name="ignition::gazebo::systems::JointStatePublisher"/>
+    </gazebo>
+  </xacro:if>
+  <xacro:if value="${'$(arg ignition_gazebo)' == 'false'}">
+    <!-- ros_control plugin -->
+    <gazebo>
+      <plugin name="gazebo_ros_control" filename="libgazebo_ros_control.so">
+        <robotNamespace>/go1_gazebo</robotNamespace>
+        <robotSimType>gazebo_ros_control/DefaultRobotHWSim</robotSimType>
+      </plugin>
+    </gazebo>
+    <!-- Show the trajectory of trunk center. -->
+    <gazebo>
+      <plugin name="3dplot" filename="libLinkPlot3DPlugin.so">
+        <frequency>10</frequency>
+        <plot>
+          <link>base</link>
+          <pose>0 0 0 0 0 0</pose>
+          <material>Gazebo/Yellow</material>
+        </plot>
+      </plugin>
+    </gazebo>
+    <!-- Show the trajectory of foot. You can add another trajectory about another foot. -->
+    <!-- <gazebo>
+            <plugin name="3dplot" filename="libLinkPlot3DPlugin.so">
+                <frequency>100</frequency>
+                <plot>
+                    <link>FL_foot</link>
+                    <pose>0 0 0 0 0 0</pose>
+                    <material>Gazebo/Green</material>
+                </plot>
+            </plugin>
+        </gazebo> -->
+    <gazebo>
+      <plugin filename="libgazebo_ros_force.so" name="gazebo_ros_force">
+        <bodyName>trunk</bodyName>
+        <topicName>/apply_force/trunk</topicName>
+      </plugin>
+    </gazebo>
+  </xacro:if>
   <gazebo reference="imu_link">
     <gravity>true</gravity>
@@ -43,61 +51,21 @@
       <visualize>true</visualize>
       <topic>__default_topic__</topic>
-      <plugin filename="libgazebo_ros_imu_sensor.so" name="imu_plugin">
-        <topicName>trunk_imu</topicName>
-        <bodyName>imu_link</bodyName>
-        <updateRateHZ>1000.0</updateRateHZ>
-        <gaussianNoise>0.0</gaussianNoise>
-        <xyzOffset>0 0 0</xyzOffset>
-        <rpyOffset>0 0 0</rpyOffset>
-        <frameName>imu_link</frameName>
-      </plugin>
+      <xacro:if value="${'$(arg ignition_gazebo)' == 'false'}">
+        <plugin filename="libgazebo_ros_imu_sensor.so" name="imu_plugin">
+          <topicName>trunk_imu</topicName>
+          <bodyName>imu_link</bodyName>
+          <updateRateHZ>1000.0</updateRateHZ>
+          <gaussianNoise>0.0</gaussianNoise>
+          <xyzOffset>0 0 0</xyzOffset>
+          <rpyOffset>0 0 0</rpyOffset>
+          <frameName>imu_link</frameName>
+        </plugin>
+      </xacro:if>
       <pose>0 0 0 0 0 0</pose>
     </sensor>
   </gazebo>
   <!-- Depth camera -->
-  <!-- <gazebo>
-        <plugin name="camera_plugin" filename="libgazebo_ros_openni_kinect.so">
-            <baseline>0.025</baseline>
-            <always_on>true</always_on>
-            <updateRate>0.0</updateRate>
-            <cameraName>unitree_camera_left</cameraName>
-            <frameName>depthCamera_link_left</frameName>
-            <imageTopicName>rgb/imageRaw_left</imageTopicName>
-            <depthImageTopicName>depth/imageRaw_left</depthImageTopicName>
-            <pointCloudTopicName>depth/points_left</pointCloudTopicName>
-            <cameraInfoTopicName>rgb/cameraInfo_left</cameraInfoTopicName>
-            <depthImageCameraInfoTopicName>depth/cameraInfo_left</depthImageCameraInfoTopicName>
-            <pointCloudCutoff>0.1</pointCloudCutoff>
-            <pointCloudCutoffMax>1.5</pointCloudCutoffMax>
-            <distortionK1>0.0</distortionK1>
-            <distortionK2>0.0</distortionK2>
-            <distortionK3>0.0</distortionK3>
-            <distortionT1>0.0</distortionT1>
-            <distortionT2>0.0</distortionT2>
-            <CxPrime>0.0</CxPrime>
-            <Cx>0.0045</Cx>
-            <Cy>0.0039</Cy>
-            <focalLength>0.004</focalLength>
-            <hackBaseline>0.0</hackBaseline>
-        </plugin>
-    </gazebo> -->
-  <!-- <gazebo reference="depthCamera_link_left">
-        <sensor name="unitree_camera_left" type="depth_camera">
-            <update_rate>16</update_rate>
-            <always_on>true</always_on>
-            <visualize>true</visualize>
-            <camera>
-                <horizontal_fov>2.094</horizontal_fov>
-                <image>
-                    <width>928</width>
-                    <height>800</height>
-                    <format>R8G8B8</format>
-                </image>
-                <depth_camera></depth_camera>
-                <clip>
-                    <near>0.1</near>
-                    <far>100</far>
-                </clip>
-            </camera>
+  <xacro:if value="${'$(arg ignition_gazebo)' == 'false'}">
+    <!-- <gazebo>
             <plugin name="camera_plugin" filename="libgazebo_ros_openni_kinect.so">
                 <baseline>0.025</baseline>
@@ -124,4 +92,50 @@
                 <hackBaseline>0.0</hackBaseline>
             </plugin>
+        </gazebo> -->
+  </xacro:if>
+  <!-- <gazebo reference="depthCamera_link_left">
+        <sensor name="unitree_camera_left" type="depth_camera">
+            <update_rate>16</update_rate>
+            <always_on>true</always_on>
+            <visualize>true</visualize>
+            <camera>
+                <horizontal_fov>2.094</horizontal_fov>
+                <image>
+                    <width>928</width>
+                    <height>800</height>
+                    <format>R8G8B8</format>
+                </image>
+                <depth_camera></depth_camera>
+                <clip>
+                    <near>0.1</near>
+                    <far>100</far>
+                </clip>
+            </camera>
+            <xacro:if value="${'$(arg ignition_gazebo)' == 'false'}">
+                <plugin name="camera_plugin" filename="libgazebo_ros_openni_kinect.so">
+                    <baseline>0.025</baseline>
+                    <always_on>true</always_on>
+                    <updateRate>0.0</updateRate>
+                    <cameraName>unitree_camera_left</cameraName>
+                    <frameName>depthCamera_link_left</frameName>
+                    <imageTopicName>rgb/imageRaw_left</imageTopicName>
+                    <depthImageTopicName>depth/imageRaw_left</depthImageTopicName>
+                    <pointCloudTopicName>depth/points_left</pointCloudTopicName>
+                    <cameraInfoTopicName>rgb/cameraInfo_left</cameraInfoTopicName>
+                    <depthImageCameraInfoTopicName>depth/cameraInfo_left</depthImageCameraInfoTopicName>
+                    <pointCloudCutoff>0.1</pointCloudCutoff>
+                    <pointCloudCutoffMax>1.5</pointCloudCutoffMax>
+                    <distortionK1>0.0</distortionK1>
+                    <distortionK2>0.0</distortionK2>
+                    <distortionK3>0.0</distortionK3>
+                    <distortionT1>0.0</distortionT1>
+                    <distortionT2>0.0</distortionT2>
+                    <CxPrime>0.0</CxPrime>
+                    <Cx>0.0045</Cx>
+                    <Cy>0.0039</Cy>
+                    <focalLength>0.004</focalLength>
+                    <hackBaseline>0.0</hackBaseline>
+                </plugin>
+            </xacro:if>
         </sensor>
     </gazebo> -->
@@ -141,28 +155,30 @@
         </clip>
       </camera>
-      <plugin name="camera_link_controller" filename="libgazebo_ros_openni_kinect.so">
-        <baseline>0.2</baseline>
-        <alwaysOn>true</alwaysOn>
-        <updateRate>1.0</updateRate>
-        <cameraName>camera_link_ir</cameraName>
-        <imageTopicName>/camera_link/color/image_raw</imageTopicName>
-        <cameraInfoTopicName>/camera_link/color/camera_info</cameraInfoTopicName>
-        <depthImageTopicName>/camera_link/depth/image_raw</depthImageTopicName>
-        <depthImageInfoTopicName>/camera_link/depth/camera_info</depthImageInfoTopicName>
-        <pointCloudTopicName>/camera_link/depth/points</pointCloudTopicName>
-        <frameName>depthCamera_link_left</frameName>
-        <pointCloudCutoff>0.5</pointCloudCutoff>
-        <pointCloudCutoffMax>3.0</pointCloudCutoffMax>
-        <distortionK1>0.00000001</distortionK1>
-        <distortionK2>0.00000001</distortionK2>
-        <distortionK3>0.00000001</distortionK3>
-        <distortionT1>0.00000001</distortionT1>
-        <distortionT2>0.00000001</distortionT2>
-        <CxPrime>0</CxPrime>
-        <Cx>0</Cx>
-        <Cy>0</Cy>
-        <focalLength>0</focalLength>
-        <hackBaseline>0</hackBaseline>
-      </plugin>
+      <xacro:if value="${'$(arg ignition_gazebo)' == 'false'}">
+        <plugin name="camera_link_controller" filename="libgazebo_ros_openni_kinect.so">
+          <baseline>0.2</baseline>
+          <alwaysOn>true</alwaysOn>
+          <updateRate>1.0</updateRate>
+          <cameraName>camera_link_ir</cameraName>
+          <imageTopicName>/camera_link/color/image_raw</imageTopicName>
+          <cameraInfoTopicName>/camera_link/color/camera_info</cameraInfoTopicName>
+          <depthImageTopicName>/camera_link/depth/image_raw</depthImageTopicName>
+          <depthImageInfoTopicName>/camera_link/depth/camera_info</depthImageInfoTopicName>
+          <pointCloudTopicName>/camera_link/depth/points</pointCloudTopicName>
+          <frameName>depthCamera_link_left</frameName>
+          <pointCloudCutoff>0.5</pointCloudCutoff>
+          <pointCloudCutoffMax>3.0</pointCloudCutoffMax>
+          <distortionK1>0.00000001</distortionK1>
+          <distortionK2>0.00000001</distortionK2>
+          <distortionK3>0.00000001</distortionK3>
+          <distortionT1>0.00000001</distortionT1>
+          <distortionT2>0.00000001</distortionT2>
+          <CxPrime>0</CxPrime>
+          <Cx>0</Cx>
+          <Cy>0</Cy>
+          <focalLength>0</focalLength>
+          <hackBaseline>0</hackBaseline>
+        </plugin>
+      </xacro:if>
     </sensor>
   </gazebo>
@@ -171,5 +187,7 @@
     <sensor name="FR_foot_contact" type="contact">
       <update_rate>100</update_rate>
-      <plugin name="contactPlugin" filename="libunitreeFootContactPlugin.so"/>
+      <xacro:if value="${'$(arg ignition_gazebo)' == 'false'}">
+        <plugin name="contactPlugin" filename="libunitreeFootContactPlugin.so"/>
+      </xacro:if>
       <contact>
         <collision>FR_calf_fixed_joint_lump__FR_foot_collision_1</collision>
@@ -180,5 +198,7 @@
     <sensor name="FL_foot_contact" type="contact">
       <update_rate>100</update_rate>
-      <plugin name="contactPlugin" filename="libunitreeFootContactPlugin.so"/>
+      <xacro:if value="${'$(arg ignition_gazebo)' == 'false'}">
+        <plugin name="contactPlugin" filename="libunitreeFootContactPlugin.so"/>
+      </xacro:if>
       <contact>
         <collision>FL_calf_fixed_joint_lump__FL_foot_collision_1</collision>
@@ -189,5 +209,7 @@
     <sensor name="RR_foot_contact" type="contact">
       <update_rate>100</update_rate>
-      <plugin name="contactPlugin" filename="libunitreeFootContactPlugin.so"/>
+      <xacro:if value="${'$(arg ignition_gazebo)' == 'false'}">
+        <plugin name="contactPlugin" filename="libunitreeFootContactPlugin.so"/>
+      </xacro:if>
       <contact>
         <collision>RR_calf_fixed_joint_lump__RR_foot_collision_1</collision>
@@ -198,5 +220,7 @@
     <sensor name="RL_foot_contact" type="contact">
       <update_rate>100</update_rate>
-      <plugin name="contactPlugin" filename="libunitreeFootContactPlugin.so"/>
+      <xacro:if value="${'$(arg ignition_gazebo)' == 'false'}">
+        <plugin name="contactPlugin" filename="libunitreeFootContactPlugin.so"/>
+      </xacro:if>
       <contact>
         <collision>RL_calf_fixed_joint_lump__RL_foot_collision_1</collision>
@@ -205,32 +229,34 @@
   </gazebo>
   <!-- Visualization of Foot contacts. -->
-  <gazebo reference="FR_foot">
-    <visual>
-      <plugin name="drawForcePlugin" filename="libunitreeDrawForcePlugin.so">
-        <topicName>FR_foot_contact</topicName>
-      </plugin>
-    </visual>
-  </gazebo>
-  <gazebo reference="FL_foot">
-    <visual>
-      <plugin name="drawForcePlugin" filename="libunitreeDrawForcePlugin.so">
-        <topicName>FL_foot_contact</topicName>
-      </plugin>
-    </visual>
-  </gazebo>
-  <gazebo reference="RR_foot">
-    <visual>
-      <plugin name="drawForcePlugin" filename="libunitreeDrawForcePlugin.so">
-        <topicName>RR_foot_contact</topicName>
-      </plugin>
-    </visual>
-  </gazebo>
-  <gazebo reference="RL_foot">
-    <visual>
-      <plugin name="drawForcePlugin" filename="libunitreeDrawForcePlugin.so">
-        <topicName>RL_foot_contact</topicName>
-      </plugin>
-    </visual>
-  </gazebo>
+  <xacro:if value="${'$(arg ignition_gazebo)' == 'false'}">
+    <gazebo reference="FR_foot">
+      <visual>
+        <plugin name="drawForcePlugin" filename="libunitreeDrawForcePlugin.so">
+          <topicName>FR_foot_contact</topicName>
+        </plugin>
+      </visual>
+    </gazebo>
+    <gazebo reference="FL_foot">
+      <visual>
+        <plugin name="drawForcePlugin" filename="libunitreeDrawForcePlugin.so">
+          <topicName>FL_foot_contact</topicName>
+        </plugin>
+      </visual>
+    </gazebo>
+    <gazebo reference="RR_foot">
+      <visual>
+        <plugin name="drawForcePlugin" filename="libunitreeDrawForcePlugin.so">
+          <topicName>RR_foot_contact</topicName>
+        </plugin>
+      </visual>
+    </gazebo>
+    <gazebo reference="RL_foot">
+      <visual>
+        <plugin name="drawForcePlugin" filename="libunitreeDrawForcePlugin.so">
+          <topicName>RL_foot_contact</topicName>
+        </plugin>
+      </visual>
+    </gazebo>
+  </xacro:if>
   <gazebo reference="base_link">
     <material>Gazebo/Green</material>

File: robots/go1_description/models/urdf/unitree_go1.urdf.xacro (robot description, xacro)
@@ -1,4 +1,4 @@
 <?xml version="1.0"?>
-<robot xmlns:xacro="http://www.ros.org/wiki/xacro" name="go1_description">
+<robot xmlns:xacro="http://www.ros.org/wiki/xacro" name="unitree_go1">
   <xacro:include filename="$(find go1_description)/models/urdf/const.xacro"/>
   <xacro:include filename="$(find go1_description)/models/urdf/materials.xacro"/>
