Commit message: refactored the properties of gazebo robot model
Signed-off-by: NaokiTakahashi <naoki.takahashi060@gmail.com>

File: robots/go1_description/models/urdf/const.xacro (robot description, xacro)
@@ -90,3 +90,11 @@
   <!-- foot -->
   <xacro:property name="foot_mass" value="0.06"/>
+  <!-- Gazebo simulation properties -->
+  <xacro:property name="leg_link_kp" value="100.0"/>
+  <xacro:property name="leg_link_kd" value="1.0"/>
+  <xacro:property name="enable_self_collision_check" value="true"/>
+  <xacro:property name="default_link_mu1" value="0.2"/>
+  <xacro:property name="default_link_mu2" value="0.2"/>
+  <xacro:property name="foot_link_mu1" value="0.6"/>
+  <xacro:property name="foot_link_mu2" value="0.6"/>
 </robot>

File: robots/go1_description/models/urdf/depthCamera.xacro (robot description, xacro)
@@ -33,50 +33,8 @@
     </joint>
     <link name="camera_optical_${name}">
-        </link>
-    <gazebo reference="camera_${name}">
-      <!-- <material>Gazebo/Black</material> -->
-      <sensor name="camera_${name}_camera" type="depth">
-        <update_rate>16</update_rate>
-        <camera>
-          <horizontal_fov>2.094</horizontal_fov>
-          <image>
-            <width>928</width>
-            <height>800</height>
-            <format>R8G8B8</format>
-          </image>
-          <clip>
-            <near>0.1</near>
-            <far>5</far>
-          </clip>
-        </camera>
-        <xacro:if value="${'$(arg ignition_gazebo)' == 'false'}">
-          <plugin name="camera_${name}_controller" filename="libgazebo_ros_openni_kinect.so">
-            <baseline>0.025</baseline>
-            <alwaysOn>true</alwaysOn>
-            <updateRate>0.0</updateRate>
-            <cameraName>camera_${name}_ir</cameraName>
-            <imageTopicName>/camera_${name}/color/image_raw</imageTopicName>
-            <cameraInfoTopicName>/camera_${name}/color/camera_info</cameraInfoTopicName>
-            <depthImageTopicName>/camera_${name}/depth/image_raw</depthImageTopicName>
-            <depthImageInfoTopicName>/camera_${name}/depth/camera_info</depthImageInfoTopicName>
-            <!-- <pointCloudTopicName>/camera_${name}/depth/points</pointCloudTopicName> -->
-            <pointCloudTopicName>/cam${camID}/point_cloud_${name}</pointCloudTopicName>
-            <frameName>camera_optical_${name}</frameName>
-            <pointCloudCutoff>0.1</pointCloudCutoff>
-            <pointCloudCutoffMax>1.5</pointCloudCutoffMax>
-            <distortionK1>0.0</distortionK1>
-            <distortionK2>0.0</distortionK2>
-            <distortionK3>0.0</distortionK3>
-            <distortionT1>0.0</distortionT1>
-            <distortionT2>0.0</distortionT2>
-            <CxPrime>0</CxPrime>
-            <Cx>0.0045</Cx>
-            <Cy>0.0039</Cy>
-            <focalLength>0</focalLength>
-            <hackBaseline>0</hackBaseline>
-          </plugin>
-        </xacro:if>
-      </sensor>
-    </gazebo>
+    </link>
+    <xacro:if value="$(arg use_gazebo)">
+      <xacro:depth_camera_gazebo_configulation name="${name}"/>
+    </xacro:if>
   </xacro:macro>
 </robot>

File: robots/go1_description/models/urdf/gazebo.xacro (robot description, xacro)
@@ -1,8 +1,6 @@
 <?xml version="1.0"?>
 <robot xmlns:xacro="http://www.ros.org/wiki/xacro">
-  <xacro:arg name="ignition_gazebo" default="true"/>
-  <xacro:arg name="enable_sensors_plugin" default="false"/>
-  <xacro:if value="$(arg ignition_gazebo)">
-    <gazebo>
+  <gazebo>
+    <xacro:if value="$(arg ignition_gazebo)">
       <plugin filename="ignition-gazebo-joint-state-publisher-system" name="ignition::gazebo::systems::JointStatePublisher"/>
       <plugin filename="ignition-gazebo-contact-system" name="ignition::gazebo::systems::Contact"/>
@@ -11,55 +9,47 @@
         <plugin filename="ignition-gazebo-sensors-system" name="ignition::gazebo::systems::Sensors"/>
       </xacro:if>
-    </gazebo>
-  </xacro:if>
-  <xacro:if value="${'$(arg ignition_gazebo)' == 'false'}">
-    <!-- ros_control plugin -->
-    <gazebo>
+    </xacro:if>
+    <xacro:unless value="$(arg ignition_gazebo)">
+      <!-- ros_control plugin -->
       <plugin name="gazebo_ros_control" filename="libgazebo_ros_control.so">
         <robotNamespace>/go1_gazebo</robotNamespace>
         <robotSimType>gazebo_ros_control/DefaultRobotHWSim</robotSimType>
       </plugin>
-    </gazebo>
-    <!-- Show the trajectory of trunk center. -->
-    <gazebo>
+      <!-- Show the trajectory of trunk center. -->
       <plugin name="3dplot" filename="libLinkPlot3DPlugin.so">
         <frequency>10</frequency>
         <plot>
-          <link>base</link>
+          <link>base_link</link>
           <pose>0 0 0 0 0 0</pose>
           <material>Gazebo/Yellow</material>
         </plot>
       </plugin>
-    </gazebo>
-    <!-- Show the trajectory of foot. You can add another trajectory about another foot. -->
-    <!-- <gazebo>
-            <plugin name="3dplot" filename="libLinkPlot3DPlugin.so">
-                <frequency>100</frequency>
-                <plot>
-                    <link>FL_foot</link>
-                    <pose>0 0 0 0 0 0</pose>
-                    <material>Gazebo/Green</material>
-                </plot>
-            </plugin>
-        </gazebo> -->
-    <gazebo>
+      <!-- Show the trajectory of foot. You can add another trajectory about another foot. -->
+      <plugin name="3dplot" filename="libLinkPlot3DPlugin.so">
+        <frequency>100</frequency>
+        <plot>
+          <link>FL_foot</link>
+          <pose>0 0 0 0 0 0</pose>
+          <material>Gazebo/Green</material>
+        </plot>
+      </plugin>
       <plugin filename="libgazebo_ros_force.so" name="gazebo_ros_force">
         <bodyName>trunk</bodyName>
         <topicName>/apply_force/trunk</topicName>
       </plugin>
-    </gazebo>
-  </xacro:if>
+    </xacro:unless>
+  </gazebo>
   <gazebo reference="imu_link">
     <gravity>true</gravity>
     <sensor name="imu_sensor" type="imu">
       <always_on>true</always_on>
-      <update_rate>1000</update_rate>
-      <visualize>true</visualize>
-      <xacro:if value="${'$(arg ignition_gazebo)' == 'false'}">
+      <update_rate>100</update_rate>
+      <visualize>false</visualize>
+      <xacro:unless value="$(arg ignition_gazebo)">
         <topic>__default_topic__</topic>
         <plugin filename="libgazebo_ros_imu_sensor.so" name="imu_plugin">
           <topicName>trunk_imu</topicName>
           <bodyName>imu_link</bodyName>
-          <updateRateHZ>1000.0</updateRateHZ>
+          <updateRateHZ>100.0</updateRateHZ>
           <gaussianNoise>0.0</gaussianNoise>
           <xyzOffset>0 0 0</xyzOffset>
@@ -67,200 +57,181 @@
           <frameName>imu_link</frameName>
         </plugin>
-      </xacro:if>
+      </xacro:unless>
       <pose>0 0 0 0 0 0</pose>
     </sensor>
   </gazebo>
-  <!-- Foot contacts. -->
-  <gazebo reference="FR_calf">
-    <sensor name="FR_foot_contact" type="contact">
-      <update_rate>100</update_rate>
-      <always_on>true</always_on>
-      <xacro:if value="${'$(arg ignition_gazebo)' == 'false'}">
-        <plugin name="contactPlugin" filename="libunitreeFootContactPlugin.so"/>
-      </xacro:if>
-      <contact>
-        <collision>FR_calf_fixed_joint_lump__FR_foot_collision_1</collision>
-      </contact>
-    </sensor>
-  </gazebo>
-  <gazebo reference="FL_calf">
-    <sensor name="FL_foot_contact" type="contact">
-      <update_rate>100</update_rate>
-      <always_on>true</always_on>
-      <xacro:if value="${'$(arg ignition_gazebo)' == 'false'}">
-        <plugin name="contactPlugin" filename="libunitreeFootContactPlugin.so"/>
-      </xacro:if>
-      <contact>
-        <collision>FL_calf_fixed_joint_lump__FL_foot_collision_1</collision>
-      </contact>
-    </sensor>
-  </gazebo>
-  <gazebo reference="RR_calf">
-    <sensor name="RR_foot_contact" type="contact">
-      <update_rate>100</update_rate>
-      <always_on>true</always_on>
-      <xacro:if value="${'$(arg ignition_gazebo)' == 'false'}">
-        <plugin name="contactPlugin" filename="libunitreeFootContactPlugin.so"/>
-      </xacro:if>
-      <contact>
-        <collision>RR_calf_fixed_joint_lump__RR_foot_collision_1</collision>
-      </contact>
-    </sensor>
-  </gazebo>
-  <gazebo reference="RL_calf">
-    <sensor name="RL_foot_contact" type="contact">
-      <update_rate>100</update_rate>
-      <always_on>true</always_on>
-      <xacro:if value="${'$(arg ignition_gazebo)' == 'false'}">
-        <plugin name="contactPlugin" filename="libunitreeFootContactPlugin.so"/>
-      </xacro:if>
-      <contact>
-        <collision>RL_calf_fixed_joint_lump__RL_foot_collision_1</collision>
-      </contact>
-    </sensor>
-  </gazebo>
-  <!-- Visualization of Foot contacts. -->
-  <xacro:if value="${'$(arg ignition_gazebo)' == 'false'}">
-    <gazebo reference="FR_foot">
-      <visual>
-        <plugin name="drawForcePlugin" filename="libunitreeDrawForcePlugin.so">
-          <topicName>FR_foot_contact</topicName>
-        </plugin>
-      </visual>
-    </gazebo>
-    <gazebo reference="FL_foot">
-      <visual>
-        <plugin name="drawForcePlugin" filename="libunitreeDrawForcePlugin.so">
-          <topicName>FL_foot_contact</topicName>
-        </plugin>
-      </visual>
-    </gazebo>
-    <gazebo reference="RR_foot">
-      <visual>
-        <plugin name="drawForcePlugin" filename="libunitreeDrawForcePlugin.so">
-          <topicName>RR_foot_contact</topicName>
-        </plugin>
-      </visual>
-    </gazebo>
-    <gazebo reference="RL_foot">
-      <visual>
-        <plugin name="drawForcePlugin" filename="libunitreeDrawForcePlugin.so">
-          <topicName>RL_foot_contact</topicName>
-        </plugin>
-      </visual>
-    </gazebo>
-  </xacro:if>
   <gazebo reference="base_link">
     <turnGravityOff>false</turnGravityOff>
   </gazebo>
   <gazebo reference="trunk">
-    <mu1>0.2</mu1>
-    <mu2>0.2</mu2>
-    <kp value="1000000.0"/>
-    <kd value="1.0"/>
+    <mu1>
+      ${default_link_mu1}
+    </mu1>
+    <mu2>
+      ${default_link_mu2}
+    </mu2>
+    <kp value="${leg_link_kp}"/>
+    <kd value="${leg_link_kd}"/>
   </gazebo>
   <gazebo reference="stick_link">
-    <mu1>0.2</mu1>
-    <mu2>0.2</mu2>
-  </gazebo>
-  <gazebo reference="imu_link">
-    <mu1>0.2</mu1>
-    <mu2>0.2</mu2>
-  </gazebo>
-  <!-- FL leg -->
-  <gazebo reference="FL_hip">
-    <mu1>0.2</mu1>
-    <mu2>0.2</mu2>
-  </gazebo>
-  <gazebo reference="FL_thigh">
-    <mu1>0.2</mu1>
-    <mu2>0.2</mu2>
-    <self_collide>1</self_collide>
-    <kp value="1000000.0"/>
-    <kd value="1.0"/>
-  </gazebo>
-  <gazebo reference="FL_calf">
-    <mu1>0.2</mu1>
-    <mu2>0.2</mu2>
-    <self_collide>1</self_collide>
-  </gazebo>
-  <gazebo reference="FL_foot">
-    <mu1>0.6</mu1>
-    <mu2>0.6</mu2>
-    <self_collide>1</self_collide>
-    <kp value="1000000.0"/>
-    <kd value="1.0"/>
-  </gazebo>
-  <!-- FR leg -->
-  <gazebo reference="FR_hip">
-    <mu1>0.2</mu1>
-    <mu2>0.2</mu2>
-  </gazebo>
-  <gazebo reference="FR_thigh">
-    <mu1>0.2</mu1>
-    <mu2>0.2</mu2>
-    <self_collide>1</self_collide>
-    <kp value="1000000.0"/>
-    <kd value="1.0"/>
-  </gazebo>
-  <gazebo reference="FR_calf">
-    <mu1>0.2</mu1>
-    <mu2>0.2</mu2>
-    <self_collide>1</self_collide>
-  </gazebo>
-  <gazebo reference="FR_foot">
-    <mu1>0.6</mu1>
-    <mu2>0.6</mu2>
-    <self_collide>1</self_collide>
-    <kp value="1000000.0"/>
-    <kd value="1.0"/>
-  </gazebo>
-  <!-- RL leg -->
-  <gazebo reference="RL_hip">
-    <mu1>0.2</mu1>
-    <mu2>0.2</mu2>
-  </gazebo>
-  <gazebo reference="RL_thigh">
-    <mu1>0.2</mu1>
-    <mu2>0.2</mu2>
-    <self_collide>1</self_collide>
-    <kp value="1000000.0"/>
-    <kd value="1.0"/>
-  </gazebo>
-  <gazebo reference="RL_calf">
-    <mu1>0.2</mu1>
-    <mu2>0.2</mu2>
-    <self_collide>1</self_collide>
-  </gazebo>
-  <gazebo reference="RL_foot">
-    <mu1>0.6</mu1>
-    <mu2>0.6</mu2>
-    <self_collide>1</self_collide>
-    <kp value="1000000.0"/>
-    <kd value="1.0"/>
-  </gazebo>
-  <!-- RR leg -->
-  <gazebo reference="RR_hip">
-    <mu1>0.2</mu1>
-    <mu2>0.2</mu2>
-  </gazebo>
-  <gazebo reference="RR_thigh">
-    <mu1>0.2</mu1>
-    <mu2>0.2</mu2>
-    <self_collide>1</self_collide>
-    <kp value="1000000.0"/>
-    <kd value="1.0"/>
-  </gazebo>
-  <gazebo reference="RR_calf">
-    <mu1>0.2</mu1>
-    <mu2>0.2</mu2>
-    <self_collide>1</self_collide>
-  </gazebo>
-  <gazebo reference="RR_foot">
-    <mu1>0.6</mu1>
-    <mu2>0.6</mu2>
-    <self_collide>1</self_collide>
-    <kp value="1000000.0"/>
-    <kd value="1.0"/>
-  </gazebo>
+    <mu1>
+      ${default_link_mu1}
+    </mu1>
+    <mu2>
+      ${default_link_mu2}
+    </mu2>
+  </gazebo>
+  <xacro:macro name="leg_gazebo_configulation" params="name">
+    <gazebo reference="${name}_hip">
+      <mu1>
+        ${default_link_mu1}
+      </mu1>
+      <mu2>
+        ${default_link_mu2}
+      </mu2>
+      <kp value="${leg_link_kp}"/>
+      <kd value="${leg_link_kd}"/>
+      <self_collide>
+        ${enable_self_collision_check}
+      </self_collide>
+      <xacro:if value="$(arg ignition_gazebo)">
+      </xacro:if>
+      <xacro:unless value="$(arg ignition_gazebo)">
+      </xacro:unless>
+    </gazebo>
+    <gazebo reference="${name}_thigh_shoulder">
+      <mu1>
+        ${default_link_mu1}
+      </mu1>
+      <mu2>
+        ${default_link_mu2}
+      </mu2>
+      <kp value="${leg_link_kp}"/>
+      <kd value="${leg_link_kd}"/>
+      <self_collide>
+        ${enable_self_collision_check}
+      </self_collide>
+      <xacro:if value="$(arg ignition_gazebo)">
+      </xacro:if>
+      <xacro:unless value="$(arg ignition_gazebo)">
+      </xacro:unless>
+    </gazebo>
+    <gazebo reference="${name}_thigh">
+      <mu1>
+        ${default_link_mu1}
+      </mu1>
+      <mu2>
+        ${default_link_mu2}
+      </mu2>
+      <kp value="${leg_link_kp}"/>
+      <kd value="${leg_link_kd}"/>
+      <self_collide>
+        ${enable_self_collision_check}
+      </self_collide>
+      <xacro:if value="$(arg ignition_gazebo)">
+      </xacro:if>
+      <xacro:unless value="$(arg ignition_gazebo)">
+      </xacro:unless>
+    </gazebo>
+    <gazebo reference="${name}_calf">
+      <mu1>
+        ${default_link_mu1}
+      </mu1>
+      <mu2>
+        ${default_link_mu2}
+      </mu2>
+      <kp value="${leg_link_kp}"/>
+      <kd value="${leg_link_kd}"/>
+      <self_collide>
+        ${enable_self_collision_check}
+      </self_collide>
+      <!-- Foot contacts. -->
+      <sensor name="${name}_foot_contact" type="contact">
+        <update_rate>100</update_rate>
+        <always_on>true</always_on>
+        <visualize>false</visualize>
+        <xacro:unless value="$(arg ignition_gazebo)">
+          <plugin name="contactPlugin" filename="libunitreeFootContactPlugin.so"/>
+        </xacro:unless>
+        <contact>
+          <collision>
+            ${name}_calf_fixed_joint_lump__${name}_foot_collision_1
+          </collision>
+        </contact>
+      </sensor>
+      <xacro:if value="$(arg ignition_gazebo)">
+      </xacro:if>
+      <xacro:unless value="$(arg ignition_gazebo)">
+      </xacro:unless>
+    </gazebo>
+    <gazebo reference="${name}_foot">
+      <mu1>
+        ${foot_link_mu1}
+      </mu1>
+      <mu2>
+        ${foot_link_mu2}
+      </mu2>
+      <kp value="${leg_link_kp}"/>
+      <kd value="${leg_link_kd}"/>
+      <self_collide>
+        ${enable_self_collision_check}
+      </self_collide>
+      <xacro:if value="$(arg ignition_gazebo)">
+      </xacro:if>
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
File: robots/go1_description/models/urdf/leg.xacro (robot description, xacro)
@@ -133,5 +133,5 @@
           <sphere radius="${foot_radius-0.01}"/>
         </geometry>
-        <material name="silver"/>
+        <material name="black"/>
       </visual>
       <collision>
@@ -147,4 +147,7 @@
     </link>
     <xacro:leg_transmission name="${name}"/>
+    <xacro:if value="$(arg use_gazebo)">
+      <xacro:leg_gazebo_configulation name="${name}"/>
+    </xacro:if>
   </xacro:macro>
 </robot>

File: robots/go1_description/models/urdf/unitree_go1.urdf.xacro (robot description, xacro)
@@ -1,13 +1,16 @@
 <?xml version="1.0"?>
 <robot xmlns:xacro="http://www.ros.org/wiki/xacro" name="unitree_go1">
+  <xacro:arg name="use_gazebo" default="true"/>
+  <xacro:arg name="ignition_gazebo" default="true"/>
+  <!-- Enable depth camera simulation for ignition gazebo -->
+  <xacro:arg name="enable_sensors_plugin" default="false"/>
   <xacro:include filename="$(find go1_description)/models/urdf/const.xacro"/>
   <xacro:include filename="$(find go1_description)/models/urdf/materials.xacro"/>
+  <xacro:if value="$(arg use_gazebo)">
+    <xacro:include filename="$(find go1_description)/models/urdf/gazebo.xacro"/>
+  </xacro:if>
   <xacro:include filename="$(find go1_description)/models/urdf/leg.xacro"/>
-  <!-- <xacro:include filename="$(find go1_description)/models/urdf/stairs.xacro"/> -->
-  <xacro:include filename="$(find go1_description)/models/urdf/gazebo.xacro"/>
   <xacro:include filename="$(find go1_description)/models/urdf/depthCamera.xacro"/>
   <xacro:include filename="$(find go1_description)/models/urdf/ultraSound.xacro"/>
-  <!-- <xacro:include filename="$(find go1_gazebo)/launch/stairs.urdf.xacro"/> -->
-  <!-- <xacro:stairs stairs="15" xpos="0" ypos="0" zpos="0" /> -->
   <!-- Rollover Protection mode will add an additional stick on the top, use "true" or "false" to switch it. -->
   <xacro:property name="rolloverProtection" value="false"/>
