Commit message: support REP105
Signed-off-by: NaokiTakahashi <naoki.takahashi060@gmail.com>

File: robots/go1_description/models/urdf/gazebo.xacro (robot description, xacro)
@@ -233,5 +233,5 @@
         </visual>
     </gazebo>
-    <gazebo reference="base">
+    <gazebo reference="base_link">
         <material>Gazebo/Green</material>
         <turnGravityOff>false</turnGravityOff>

File: robots/go1_description/models/urdf/unitree_go1.urdf.xacro (robot description, xacro)
@@ -19,8 +19,8 @@
             <origin rpy="0 0 0" xyz="0 0 0"/>
             <parent link="world"/>
-            <child link="base"/>
+            <child link="base_link"/>
         </joint>
     </xacro:if>
-    <link name="base">
+    <link name="base_link">
         <visual>
             <origin rpy="0 0 0" xyz="0 0 0"/>
@@ -30,7 +30,7 @@
         </visual>
     </link>
-    <joint name="floating_base" type="fixed">
+    <joint name="floating_base_joint" type="fixed">
         <origin rpy="0 0 0" xyz="0 0 0"/>
-        <parent link="base"/>
+        <parent link="base_link"/>
         <child link="trunk"/>
     </joint>

Commit message: add single point gpu_lidar for ultrasound sensor
Signed-off-by: NaokiTakahashi <naoki.takahashi060@gmail.com>

File: robots/go1_description/models/urdf/gazebo.xacro (robot description, xacro)
@@ -307,3 +307,38 @@
     </gazebo>
   </xacro:macro>
+  <xacro:macro name="ultrasound_gazebo_configulation" params="name">
+    <gazebo reference="ultraSound_${name}">
+      <sensor name="ultrasound_${name}_sensor" type="gpu_lidar">
+        <always_on>true</always_on>
+        <update_rate>30</update_rate>
+        <visualize>false</visualize>
+        <lidar>
+          <scan>
+            <horizontal>
+              <samples>1</samples>
+              <resolution>1</resolution>
+              <min_angle>0</min_angle>
+              <max_angle>0</max_angle>
+            </horizontal>
+            <vertical>
+              <samples>1</samples>
+              <resolution>1</resolution>
+              <min_angle>-0.018</min_angle>
+              <max_angle>0.018</max_angle>
+            </vertical>
+          </scan>
+          <range>
+            <min>0.1</min>
+            <max>3</max>
+            <resolution>0.01</resolution>
+          </range>
+          <noise>
+            <type>gaussian</type>
+            <mean>0.1</mean>
+            <stddev>0.05</stddev>
+          </noise>
+        </lidar>
+      </sensor>
+    </gazebo>
+  </xacro:macro>
 </robot>

File: robots/go1_description/models/urdf/ultraSound.xacro (robot description, xacro)
@@ -27,4 +27,7 @@
       </inertial>
     </link>
+    <xacro:if value="$(arg use_gazebo)">
+      <xacro:ultrasound_gazebo_configulation name="${name}"/>
+    </xacro:if>
   </xacro:macro>
 </robot>
